File: Chris/Esquema circuito/Esquema circuito.kicad_sch (KiCad schematic)
At the start: 34 parts, among them J1 Screw_Terminal_01x02, J2 Screw_Terminal_01x02, M1 Bomba de agua 5V DC, Q1 IRFZ44N, Q2 PN2222A, Q3 PN2222A, Q4 IRFZ44N, Q5 BD135, Q6 PN2222A, U1 DS18B20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

Commit message: Last Commit Regionales
Parts:
- added R10: 1K, symbol Device:R
- added R9: A9013, OptoDevice:R_LDR_5.0x4.1mm_P3mm_Vertical, symbol Sensor_Optical:A9013
Connections:
- net GND: now also R10.2
- net at R2.1, R4.1: now also U12.J1_20 (GPIO14); no longer U12.J1_12 (GPIO8)
- net at D3.2 (A), D4.2 (A), D5.2 (A)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: now also R9.1
- net at U12.J3_20 (USB_D-/GPIO19): now also R10.1, R9.2
- new net: U6. (Out3), U9. (In1) (x3)
- new net: U5. (Out), U7. (VIn)
Other:
- moved on the sheet: D3, D4, D5, Q6, R1, R8, U1, U10, U2, U3, U8
